Commit message: Removed the reference to naviswarm package from the files

File: hybrid_rl_training/models/hokuyo/hokuyo.urdf.xacro (robot description, xacro)
@@ -12,5 +12,5 @@
         <origin xyz="0 0 0" rpy="0 0 0"/>
         <geometry>
-          <mesh filename="$(find naviswarm)/models/hokuyo/hokuyo.dae"/>
+          <mesh filename="$(find hybrid_rl_training)/models/hokuyo/hokuyo.dae"/>
         </geometry>
       </visual>

File: hybrid_rl_training/models/jackals/jackal_cam_depth.urdf.xacro (robot description, xacro)
@@ -222,14 +222,14 @@
   </joint>
   <!-- Bring in simulation data for Gazebo. -->
-  <xacro:include filename="$(find naviswarm)/models/jackals/jackal.gazebo" />
+  <xacro:include filename="$(find hybrid_rl_training)/models/jackals/jackal.gazebo" />
   <!-- Optional standard accessories, including their simulation data. The rendering
        of these into the final description is controlled by optenv variables, which
        default each one to off.-->
   <xacro:include filename="$(find jackal_description)/urdf/accessories.urdf.xacro" />
-  <xacro:include filename="$(find naviswarm)/models/realsense2_description/urdf/d435_depth.macro.xacro" />
+  <xacro:include filename="$(find hybrid_rl_training)/models/realsense2_description/urdf/d435_depth.macro.xacro" />
   <xacro:sensor_d435 prefix="" parent="rear_mount">
     <origin xyz="0 0 1" rpy="0 0 0"/>
   </xacro:sensor_d435>
-  <xacro:include filename="$(find naviswarm)/models/hokuyo/hokuyo.urdf.xacro"/>
+  <xacro:include filename="$(find hybrid_rl_training)/models/hokuyo/hokuyo.urdf.xacro"/>
   <xacro:sensor_hokuyo prefix="" parent="front_mount">
     <origin xyz="0 0 0.02" rpy="0 0 0"/>

File: hybrid_rl_training/models/turtlebot2/kobuki/kobuki.urdf.xacro (robot description, xacro)
@@ -7,6 +7,6 @@
  -->
 <robot name="kobuki" xmlns:xacro="http://ros.org/wiki/xacro">
-  <xacro:include filename="$(find naviswarm)/models/turtlebot2/common_properties.urdf.xacro"/>
-  <xacro:include filename="$(find naviswarm)/models/turtlebot2/kobuki/kobuki_gazebo.urdf.xacro"/>
+  <xacro:include filename="$(find hybrid_rl_training)/models/turtlebot2/common_properties.urdf.xacro"/>
+  <xacro:include filename="$(find hybrid_rl_training)/models/turtlebot2/kobuki/kobuki_gazebo.urdf.xacro"/>
   <!-- Kobuki -->
   <xacro:macro name="kobuki">

File: hybrid_rl_training/models/turtlebot2/sensors/hokuyo.urdf.xacro (robot description, xacro)
@@ -12,5 +12,5 @@
         <origin xyz="0 0 0" rpy="0 0 0"/>
         <geometry>
-          <mesh filename="$(find naviswarm)/models/hokuyo/hokuyo.dae"/>
+          <mesh filename="$(find hybrid_rl_training)/models/hokuyo/hokuyo.dae"/>
         </geometry>
       </visual>

File: hybrid_rl_training/models/turtlebot2/sensors/r200.urdf.xacro (robot description, xacro)
@@ -2,5 +2,5 @@
 <robot name="sensor_r200" xmlns:xacro="http://ros.org/wiki/xacro">
   <!--xacro:include filename="$(find navisim)/models/turtlebot2/turtlebot_gazebo.urdf.xacro"/-->
-  <xacro:include filename="$(find naviswarm)/models/turtlebot2/common_properties.urdf.xacro"/>
+  <xacro:include filename="$(find hybrid_rl_training)/models/turtlebot2/common_properties.urdf.xacro"/>
   <!-- Mount and camera parameters -->
   <xacro:property name="pole_px" value="-0.103" />

File: hybrid_rl_training/models/turtlebot2/turtlebot.urdf.xacro (robot description, xacro)
@@ -6,10 +6,10 @@
 -->
 <robot name="turtlebot" xmlns:xacro="http://ros.org/wiki/xacro">
-  <xacro:include filename="$(find naviswarm)/models/turtlebot2/common_properties.urdf.xacro" />
-  <xacro:include filename="$(find naviswarm)/models/turtlebot2/kobuki/kobuki.urdf.xacro" />
-  <xacro:include filename="$(find naviswarm)/models/turtlebot2/stacks/hexagons.urdf.xacro"/>
+  <xacro:include filename="$(find hybrid_rl_training)/models/turtlebot2/common_properties.urdf.xacro" />
+  <xacro:include filename="$(find hybrid_rl_training)/models/turtlebot2/kobuki/kobuki.urdf.xacro" />
+  <xacro:include filename="$(find hybrid_rl_training)/models/turtlebot2/stacks/hexagons.urdf.xacro"/>
   <!--sensors-->
-  <xacro:include filename="$(find naviswarm)/models/turtlebot2/sensors/hokuyo.urdf.xacro"/>
-  <xacro:include filename="$(find naviswarm)/models/turtlebot2/sensors/r200.urdf.xacro"/>
+  <xacro:include filename="$(find hybrid_rl_training)/models/turtlebot2/sensors/hokuyo.urdf.xacro"/>
+  <xacro:include filename="$(find hybrid_rl_training)/models/turtlebot2/sensors/r200.urdf.xacro"/>
   <!--xacro:include filename="$(find slam_ros)/models/urdf/sensors/asus_xtion_pro.urdf.xacro"/>
   <xacro:include filename="$(find slam_ros)/models/urdf/sensors/asus_xtion_pro_offset.urdf.xacro"/-->
